File: keyboard-left.kicad_pcb (KiCad board)
At the start: 2 copper layers, 193.3 x 144.8 mm, 330 parts, among them J1 ST-Link Clone (Optional), K1 Esc,,,,,,,,,F1, K10 !,1,,,,,,,,A2, K11 @,2,,,,,,,,A3, K12 #,3,,,,,,,,A4, K13 $,4,,,,,,,,A5, K14 %,5,,,,,,,,A6, K15 ^,6,,,,,,,,A7, K16 Tab,,,,1.5,,,,,B1, K17 Q,,,,,,,,,B2, K18 W,,,,,,,,,B3, K19 E,,,,,,,,,B4, K2 F1,,,,,,,,,F2, K20 R,,,,,,,,,B5, K21 T,,,,,,,,,B6, K22 Caps Lock,,,,1.75,,,,,C1, K23 A,,,,,,,,,C2, K24 S,,,,,,,,,C3, K25 D,,,,,,,,,C4, K26 F,,,,,,,,,C5, K27 G,,,,,,,,,C6, K28 Shift,,,,2.25,,,,,D1, K29 Z,,,,,,,,,D2, K3 F2,,,,,,,,,F3, K30 X,,,,,,,,,D3, K31 C,,,,,,,,,D4, K32 V,,,,,,,,,D5, K33 B,,,,,,,,,D6, K34 Ctrl,,,,1.25,,,,,E1, K35 Win,,,,1.25,,,,,E2, K36 Alt,,,,1.25,,,,,E3, K37 Space,,,,3.00,,,,,E4, K4 F3,,,,,,,,,F4, K5 F4,,,,,,,,,F5, K6 F5,,,,,,,,,F6, K7 F6,,,,,,,,,F7, K9 ~,`,,,,,,,,A1, Q1 AO3401A, Q2 AO3401A, Q3 AO3401A, Q4 2N7002, Q5 2N7002, Q6 MMUN2133LT1G, Q7 AO3401A, Q8 MMUN2233LT1G, SW1 SW_Push, SW10 SW_Push, SW11 SW_Push, SW12 SW_Push, SW13 SW_Push, SW14 SW_Push, SW15 SW_Push, SW16 SW_Push, SW17 SW_Push, SW18 SW_Push, SW19 SW_Push, SW2 SW_Push, SW20 SW_Push, SW21 SW_Push, SW22 SW_Push, SW23 SW_Push, SW24 SW_Push, SW25 SW_Push, SW26 SW_Push, SW27 SW_Push, SW28 SW_Push, SW29 SW_Push, SW3 SW_Push, SW30 SW_Push, SW31 SW_Push, SW32 SW_Push, SW33 SW_Push, SW34 SW_Push, SW35 SW_Push, SW36 SW_Push, SW4 SW_Push, SW5 SW_Push, SW6 SW_Push, SW7 SW_Push, SW8 SW_Push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

Commit message: Final component placements
Parts:
- moved FB10 264.6 mm to (169.7, 77.2), turned to 180 degrees
- moved DRILL10 263.4 mm to (176.0, 75.7)
- moved C11 154.3 mm to (143.8, 6.35), turned to 180 degrees
- moved R22 137.6 mm to (142.7, 39.9)
- moved U8 131.4 mm to (159.0, 36.8), turned to 90 degrees
- moved R13 130.1 mm to (175.0, 37.1), turned to 90 degrees
- moved R20 129.6 mm to (147.8, 39.9)
- moved C13 127.6 mm to (152.9, 37.6)
- moved R21 125.8 mm to (172.7, 37.1), turned to 90 degrees
- moved R19 120.5 mm to (170.4, 37.1), turned to 90 degrees
- moved R18 118.2 mm to (168.1, 37.1), turned to 90 degrees
- moved R15 117.4 mm to (152.9, 35.3)
- moved R14 116.6 mm to (152.9, 33.0)
- moved C6 116.3 mm to (158.2, 26.2), turned to 90 degrees
- moved R16 116.1 mm to (152.9, 39.9)
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
Commit message: Auto routing
Parts:
- removed BZ1: KLJ-1625, reversible-kicad-footprints:Piezo-KLJ-1625
- removed DRILL11: Drill Mountpoint, DjinnFootprints:MountingHole_3.2mm_M3_Pad_Via
- removed FB11: 4A/0805, reversible-kicad-footprints:L-0805_2012Metric
- removed K1: Esc,,,,,,,,,F1, MX_Only:MXOnly-1U-Hotswap-Antishear
- removed K10: !,1,,,,,,,,A2, MX_Only:MXOnly-1U-Hotswap-Antishear
- removed K11: @,2,,,,,,,,A3, MX_Only:MXOnly-1U-Hotswap-Antishear
- removed K12: #,3,,,,,,,,A4, MX_Only:MXOnly-1U-Hotswap-Antishear
- removed K13: $,4,,,,,,,,A5, MX_Only:MXOnly-1U-Hotswap-Antishear
- removed K14: %,5,,,,,,,,A6, MX_Only:MXOnly-1U-Hotswap-Antishear
- removed K15: ^,6,,,,,,,,A7, MX_Only:MXOnly-1U-Hotswap-Antishear
- removed K16: Tab,,,,1.5,,,,,B1, MX_Only:MXOnly-1.5U-Hotswap
- removed K17: Q,,,,,,,,,B2, MX_Only:MXOnly-1U-Hotswap-Antishear
- removed K18: W,,,,,,,,,B3, MX_Only:MXOnly-1U-Hotswap-Antishear
- removed K19: E,,,,,,,,,B4, MX_Only:MXOnly-1U-Hotswap-Antishear
- removed K2: F1,,,,,,,,,F2, MX_Only:MXOnly-1U-Hotswap-Antishear
- removed K20: R,,,,,,,,,B5, MX_Only:MXOnly-1U-Hotswap-Antishear
- removed K21: T,,,,,,,,,B6, MX_Only:MXOnly-1U-Hotswap-Antishear
- removed K22: Caps Lock,,,,1.75,,,,,C1, MX_Only:MXOnly-1.75U-Hotswap
- removed K23: A,,,,,,,,,C2, MX_Only:MXOnly-1U-Hotswap-Antishear
- removed K24: S,,,,,,,,,C3, MX_Only:MXOnly-1U-Hotswap-Antishear
- removed K25: D,,,,,,,,,C4, MX_Only:MXOnly-1U-Hotswap-Antishear
- removed K26: F,,,,,,,,,C5, MX_Only:MXOnly-1U-Hotswap-Antishear
- removed K27: G,,,,,,,,,C6, MX_Only:MXOnly-1U-Hotswap-Antishear
- removed K28: Shift,,,,2.25,,,,,D1, MX_Only:MXOnly-2.25U-Hotswap
- removed K29: Z,,,,,,,,,D2, MX_Only:MXOnly-1U-Hotswap-Antishear
- removed K3: F2,,,,,,,,,F3, MX_Only:MXOnly-1U-Hotswap-Antishear
- removed K30: X,,,,,,,,,D3, MX_Only:MXOnly-1U-Hotswap-Antishear
- removed K31: C,,,,,,,,,D4, MX_Only:MXOnly-1U-Hotswap-Antishear
- removed K32: V,,,,,,,,,D5, MX_Only:MXOnly-1U-Hotswap-Antishear
- removed K33: B,,,,,,,,,D6, MX_Only:MXOnly-1U-Hotswap-Antishear
- removed K34: Ctrl,,,,1.25,,,,,E1, MX_Only:MXOnly-1.25U-Hotswap
- removed K35: Win,,,,1.25,,,,,E2, MX_Only:MXOnly-1.25U-Hotswap
- removed K36: Alt,,,,1.25,,,,,E3, MX_Only:MXOnly-1.25U-Hotswap
- removed K37: Space,,,,3.00,,,,,E4, MX_Only:MXOnly-3U-Hotswap-ReversedStabilizers
- removed K4: F3,,,,,,,,,F4, MX_Only:MXOnly-1U-Hotswap-Antishear
- removed K5: F4,,,,,,,,,F5, MX_Only:MXOnly-1U-Hotswap-Antishear
- removed K6: F5,,,,,,,,,F6, MX_Only:MXOnly-1U-Hotswap-Antishear
- removed K7: F6,,,,,,,,,F7, MX_Only:MXOnly-1U-Hotswap-Antishear
- removed K9: ~,`,,,,,,,,A1, MX_Only:MXOnly-1U-Hotswap-Antishear
- removed LOGO1, LOGO2: QMK Logo, DjinnFootprints:QMK_PoweredBy
- removed LOGO7, LOGO8: QMK QRCode, DjinnFootprints:Djinn_QRCode_0.4mm
- removed TP1: VBUS, reversible-kicad-footprints:TestPoint
- removed TP10: COL1, reversible-kicad-footprints:TestPoint
- removed TP11: BOOT0_CHRG, reversible-kicad-footprints:TestPoint
- removed TP12: COL2, reversible-kicad-footprints:TestPoint
- removed TP13: COL3, reversible-kicad-footprints:TestPoint
- removed TP14: COMMS_A, reversible-kicad-footprints:TestPoint
- removed TP15: COL4, reversible-kicad-footprints:TestPoint
- removed TP16: COMMS_B, reversible-kicad-footprints:TestPoint
- removed TP17: COL5, reversible-kicad-footprints:TestPoint
- removed TP18: RGB_PW, reversible-kicad-footprints:TestPoint
- removed TP19: COL6, reversible-kicad-footprints:TestPoint
- removed TP2: SCK, reversible-kicad-footprints:TestPoint
- removed TP20: RGB_EN, reversible-kicad-footprints:TestPoint
- removed TP21: COL7, reversible-kicad-footprints:TestPoint
- removed TP22: RGB_D, reversible-kicad-footprints:TestPoint
- removed TP23: ROW1, reversible-kicad-footprints:TestPoint
- removed TP24: RGB_F, reversible-kicad-footprints:TestPoint
- removed TP25: ROW2, reversible-kicad-footprints:TestPoint
- removed TP26: RGB_1.5, reversible-kicad-footprints:TestPoint
- removed TP27: ROW3, reversible-kicad-footprints:TestPoint
- removed TP28: RGB_3.0, reversible-kicad-footprints:TestPoint
- removed TP29: ROW4, reversible-kicad-footprints:TestPoint
- removed TP3: 5V, reversible-kicad-footprints:TestPoint
- removed TP30: RGB_LM, reversible-kicad-footprints:TestPoint
- removed TP31: ROW5, reversible-kicad-footprints:TestPoint
- removed TP32: ROW6, reversible-kicad-footprints:TestPoint
- removed TP33: LCD_PW, reversible-kicad-footprints:TestPoint
- removed TP34: LCD_EN, reversible-kicad-footprints:TestPoint
- removed TP35: SPK_A, reversible-kicad-footprints:TestPoint
- removed TP36: LCD_CS, reversible-kicad-footprints:TestPoint
- removed TP37: SPK_B, reversible-kicad-footprints:TestPoint
- removed TP38: LCD_DC, reversible-kicad-footprints:TestPoint
- removed TP39: CC1, reversible-kicad-footprints:TestPoint
- removed TP4: MISO, reversible-kicad-footprints:TestPoint
- removed TP40: LCD_RST, reversible-kicad-footprints:TestPoint
- removed TP41: CC2, reversible-kicad-footprints:TestPoint
- removed TP42: LCD_BL, reversible-kicad-footprints:TestPoint
- removed TP44: EEP_CS, reversible-kicad-footprints:TestPoint
- removed TP45: PLUG, reversible-kicad-footprints:TestPoint
- removed TP46: FLASH_CS, reversible-kicad-footprints:TestPoint
- removed TP47: ENC_A, reversible-kicad-footprints:TestPoint
- removed TP48, TP50, TP51, TP52, TP53, TP54: GND, reversible-kicad-footprints:TestPoint
- removed TP49: ENC_B, reversible-kicad-footprints:TestPoint
- removed TP5: 3.3V, reversible-kicad-footprints:TestPoint
- removed TP56: MTX_CLK, reversible-kicad-footprints:TestPoint
- removed TP57: MTX_OE, reversible-kicad-footprints:TestPoint
- removed TP58: MTX_SERIAL, reversible-kicad-footprints:TestPoint
- removed TP59: MTX_SRCLR, reversible-kicad-footprints:TestPoint
- removed TP6: MOSI, reversible-kicad-footprints:TestPoint
- removed TP7: BRD_F, reversible-kicad-footprints:TestPoint
- removed TP8: NRST, reversible-kicad-footprints:TestPoint
- removed TP9: BOOT0, reversible-kicad-footprints:TestPoint
