File: keyboard-left.kicad_sch (KiCad schematic)
At the start: 295 parts, among them J1 ST-Link Clone (Optional), Q1 AO3401A, Q2 AO3401A, Q3 AO3401A, Q4 2N7002, Q5 2N7002, Q6 MMUN2133LT1G, Q7 AO3401A, Q8 MMUN2233LT1G, SW1 SW_Push, SW10 SW_Push, SW11 SW_Push, SW12 SW_Push, SW13 SW_Push, SW14 SW_Push, SW15 SW_Push, SW16 SW_Push, SW17 SW_Push, SW18 SW_Push, SW19 SW_Push, SW2 SW_Push, SW20 SW_Push, SW21 SW_Push, SW22 SW_Push, SW23 SW_Push, SW24 SW_Push, SW25 SW_Push, SW26 SW_Push, SW27 SW_Push, SW28 SW_Push, SW29 SW_Push, SW3 SW_Push, SW30 SW_Push, SW31 SW_Push, SW32 SW_Push, SW33 SW_Push, SW34 SW_Push, SW35 SW_Push, SW36 SW_Push, SW4 SW_Push, SW5 SW_Push, SW6 SW_Push, SW7 SW_Push, SW8 SW_Push, SW9 SW_Push, U1 STM32G474RETx, U10 W25Q32JVSSIQ, U11 74HC595, U2 STM32G474RETx, U3 AP2127K-3.3, U4 TPS2553DBVR-1, U5 LMV321, U6 AZC199-04S, U7 AZC199-04S, U8 TPS2553DBVR-1, U9 MB85RS64

Commit message: Minor progress on component grouping
Connections:
- net GND: now also C1.2, C2.2, C28.2, C3.2, C4.2, C5.2
- net SK6812_PWR: now also C1.1, C2.1, C28.1, C3.1, C4.1, C5.1
Other:
- moved on the sheet: C1, C2, C28, C3, C4, C5
Changed lines of the file:
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@@
     )
   )
-  (symbol (lib_id "Djinn-rescue:CP-Device") (at 533.4 176.53 0) (mirror y) (unit 1)
-    (in_bom yes) (on_board yes) (dnp no)
-    (property "Reference" "C1" (at 530.4028 175.3616 0)
-      (effects (font (size 1.27 1.27)) (justify left))
-    )
-    (property "Value" "100u" (at 530.4028 177.673 0)
-      (effects (font (size 1.27 1.27)) (justify left))
-    )
-    (property "Footprint" "reversible-kicad-footprints:CP_6032" (at 532.4348 180.34 0)
-      (effects (font (size 1.27 1.27)) hide)
-    )
-    (property "Datasheet" "~" (at 533.4 176.53 0)
+  (symbol (lib_id "Djinn-rescue:CP-Device") (at 528.32 176.53 0) (mirror y) (unit 1)
+    (in_bom yes) (on_board yes) (dnp no)
+    (property "Reference" "C1" (at 525.3228 175.3616 0)
+      (effects (font (size 1.27 1.27)) (justify left))
+    )
+    (property "Value" "100u" (at 525.3228 177.673 0)
+      (effects (font (size 1.27 1.27)) (justify left))
+    )
+    (property "Footprint" "reversible-kicad-footprints:CP_6032" (at 527.3548 180.34 0)
+      (effects (font (size 1.27 1.27)) hide)
+    )
+    (property "Datasheet" "~" (at 528.32 176.53 0)
       (effects (font (size 1.27 1.27)) hide)
     )
@@
     )
   )
-  (symbol (lib_id "Djinn-rescue:CP-Device") (at 521.97 176.53 0) (mirror y) (unit 1)
-    (in_bom yes) (on_board yes) (dnp no)
-    (property "Reference" "C2" (at 518.9728 175.3616 0)
-      (effects (font (size 1.27 1.27)) (justify left))
-    )
-    (property "Value" "100u" (at 518.9728 177.673 0)
-      (effects (font (size 1.27 1.27)) (justify left))
-    )
-    (property "Footprint" "reversible-kicad-footprints:CP_6032" (at 521.0048 180.34 0)
-      (effects (font (size 1.27 1.27)) hide)
-    )
-    (property "Datasheet" "~" (at 521.97 176.53 0)
+  (symbol (lib_id "Djinn-rescue:CP-Device") (at 516.89 176.53 0) (mirror y) (unit 1)
+    (in_bom yes) (on_board yes) (dnp no)
+    (property "Reference" "C2" (at 513.8928 175.3616 0)
+      (effects (font (size 1.27 1.27)) (justify left))
+    )
+    (property "Value" "100u" (at 513.8928 177.673 0)
+      (effects (font (size 1.27 1.27)) (justify left))
+    )
+    (property "Footprint" "reversible-kicad-footprints:CP_6032" (at 515.9248 180.34 0)
+      (effects (font (size 1.27 1.27)) hide)
+    )
+    (property "Datasheet" "~" (at 516.89 176.53 0)
       (effects (font (size 1.27 1.27)) hide)
     )
@@
     )
   )
-  (symbol (lib_id "Djinn-rescue:CP-Device") (at 510.54 176.53 0) (mirror y) (unit 1)
-    (in_bom yes) (on_board yes) (dnp no)
-    (property "Reference" "C3" (at 507.5428 175.3616 0)
-      (effects (font (size 1.27 1.27)) (justify left))
-    )
-    (property "Value" "100u" (at 507.5428 177.673 0)
-      (effects (font (size 1.27 1.27)) (justify left))
-    )
-    (property "Footprint" "reversible-kicad-footprints:CP_6032" (at 509.5748 180.34 0)
-      (effects (font (size 1.27 1.27)) hide)
-    )
-    (property "Datasheet" "~" (at 510.54 176.53 0)
+  (symbol (lib_id "Djinn-rescue:CP-Device") (at 505.46 176.53 0) (mirror y) (unit 1)
+    (in_bom yes) (on_board yes) (dnp no)
+    (property "Reference" "C3" (at 502.4628 175.3616 0)
+      (effects (font (size 1.27 1.27)) (justify left))
+    )
+    (property "Value" "100u" (at 502.4628 177.673 0)
+      (effects (font (size 1.27 1.27)) (justify left))
+    )
+    (property "Footprint" "reversible-kicad-footprints:CP_6032" (at 504.4948 180.34 0)
+      (effects (font (size 1.27 1.27)) hide)
+    )
+    (property "Datasheet" "~" (at 505.46 176.53 0)
       (effects (font (size 1.27 1.27)) hide)
     )
@@
     )
   )
-  (symbol (lib_id "Djinn-rescue:CP-Device") (at 499.11 176.53 0) (mirror y) (unit 1)
-    (in_bom yes) (on_board yes) (dnp no)
-    (property "Reference" "C4" (at 496.1128 175.3616 0)
-      (effects (font (size 1.27 1.27)) (justify left))
-    )
-    (property "Value" "100u" (at 496.1128 177.673 0)
-      (effects (font (size 1.27 1.27)) (justify left))
-    )
-    (property "Footprint" "reversible-kicad-footprints:CP_6032" (at 498.1448 180.34 0)
-      (effects (font (size 1.27 1.27)) hide)
-    )
-    (property "Datasheet" "~" (at 499.11 176.53 0)
+  (symbol (lib_id "Djinn-rescue:CP-Device") (at 494.03 176.53 0) (mirror y) (unit 1)
+    (in_bom yes) (on_board yes) (dnp no)
+    (property "Reference" "C4" (at 491.0328 175.3616 0)
+      (effects (font (size 1.27 1.27)) (justify left))
+    )
+    (property "Value" "100u" (at 491.0328 177.673 0)
+      (effects (font (size 1.27 1.27)) (justify left))
+    )
+    (property "Footprint" "reversible-kicad-footprints:CP_6032" (at 493.0648 180.34 0)
+      (effects (font (size 1.27 1.27)) hide)
+    )
+    (property "Datasheet" "~" (at 494.03 176.53 0)
       (effects (font (size 1.27 1.27)) hide)
     )
@@
     )
   )
-  (symbol (lib_id "Djinn-rescue:CP-Device") (at 487.68 176.53 0) (mirror y) (unit 1)
-    (in_bom yes) (on_board yes) (dnp no)
-    (property "Reference" "C5" (at 484.6828 175.3616 0)
-      (effects (font (size 1.27 1.27)) (justify left))
-    )
-    (property "Value" "100u" (at 484.6828 177.673 0)
-      (effects (font (size 1.27 1.27)) (justify left))
-    )
-    (property "Footprint" "reversible-kicad-footprints:CP_6032" (at 486.7148 180.34 0)
-      (effects (font (size 1.27 1.27)) hide)
-    )
-    (property "Datasheet" "~" (at 487.68 176.53 0)
+  (symbol (lib_id "Djinn-rescue:CP-Device") (at 482.6 176.53 0) (mirror y) (unit 1)
+    (in_bom yes) (on_board yes) (dnp no)
+    (property "Reference" "C5" (at 479.6028 175.3616 0)
+      (effects (font (size 1.27 1.27)) (justify left))
+    )
+    (property "Value" "100u" (at 479.6028 177.673 0)
+      (effects (font (size 1.27 1.27)) (justify left))
+    )
+    (property "Footprint" "reversible-kicad-footprints:CP_6032" (at 481.6348 180.34 0)
+      (effects (font (size 1.27 1.27)) hide)
+    )
+    (property "Datasheet" "~" (at 482.6 176.53 0)
       (effects (font (size 1.27 1.27)) hide)
     )
@@
     )
   )
-  (symbol (lib_id "Djinn-rescue:CP-Device") (at 476.25 176.53 0) (mirror y) (unit 1)
-    (in_bom yes) (on_board yes) (dnp no)
-    (property "Reference" "C28" (at 473.2528 175.3616 0)
-      (effects (font (size 1.27 1.27)) (justify left))
-    )
-    (property "Value" "100u" (at 473.2528 177.673 0)
-      (effects (font (size 1.27 1.27)) (justify left))
-    )
-    (property "Footprint" "reversible-kicad-footprints:CP_6032" (at 475.2848 180.34 0)
-      (effects (font (size 1.27 1.27)) hide)
-    )
-    (property "Datasheet" "~" (at 476.25 176.53 0)
-      (effects (font (size 1.27 1.27)) hide)
-    )
+  (symbol (lib_id "Djinn-rescue:CP-Device") (at 471.17 176.53 0) (mirror y) (unit 1)
+    (in_bom yes) (on_board yes) (dnp no)
+    (property "Reference" "C28" (at 468.1728 175.3616 0)
+      (effects (font (size 1.27 1.27)) (justify left))
+    )
+    (property "Value" "100u" (at 468.1728 177.673 0)
+      (effects (font (size 1.27 1.27)) (justify left))
+    )
+    (property "Footprint" "reversible-kicad-footprints:CP_6032" (at 470.2048 180.34 0)
+      (effects (font (size 1.27 1.27)) hide)
+    )
+    (property "Datasheet" "~" (at 471.17 176.53 0)
+      (effects (font (size 1.27 1.27)) hide)
+    )

Commit message: More component groupings
Parts:
- SPLIT1, USB1: footprint reversible-kicad-footprints:HRO-TYPE-C-31-M-12-HandSoldering-NoSBU -> Type-C.pretty-master:HRO-TYPE-C-31-M-12-HandSoldering
Changed lines of the file:
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@@
       (effects (font (size 1.27 1.27)))
     )
-    (property "Footprint" "reversible-kicad-footprints:HRO-TYPE-C-31-M-12-HandSoldering-NoSBU" (at 91.44 308.61 0)
+    (property "Footprint" "Type-C.pretty-master:HRO-TYPE-C-31-M-12-HandSoldering" (at 91.44 308.61 0)
       (effects (font (size 1.27 1.27)) hide)
     )
@@
       (effects (font (size 1.27 1.27)))
     )
-    (property "Footprint" "reversible-kicad-footprints:HRO-TYPE-C-31-M-12-HandSoldering-NoSBU" (at 789.94 311.15 0)
+    (property "Footprint" "Type-C.pretty-master:HRO-TYPE-C-31-M-12-HandSoldering" (at 789.94 311.15 0)
       (effects (font (size 1.27 1.27)) hide)
     )

Commit message: Pre-repositioning MCU
Connections:
- net EEP_CS: now also U1.2 (PC13), U2.2 (PC13); no longer U1.58 (PB5), U2.58 (PB5)
- new net: U1.58 (PB5), U2.58 (PB5)
- no-connect marks 11 -> 18
Changed lines of the file:
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@@
   (junction (at 144.78 321.31) (diameter 0) (color 0 0 0 0)
   )
-  (junction (at 518.16 342.9) (diameter 0) (color 0 0 0 0)
-  )
   (junction (at 520.7 53.34) (diameter 0) (color 0 0 0 0)
   )
@@
   (junction (at 285.75 90.17) (diameter 0) (color 0 0 0 0)
   )
+  (junction (at 589.28 320.04) (diameter 0) (color 0 0 0 0)
+  )
   (junction (at 533.4 220.98) (diameter 0) (color 0 0 0 0)
   )
@@
   (no_connect (at 427.99 521.97))
   (no_connect (at 199.39 410.21))
+  (no_connect (at 518.16 289.56))
+  (no_connect (at 518.16 294.64))
   (no_connect (at 199.39 405.13))
   (no_connect (at 212.09 410.21))
+  (no_connect (at 518.16 292.1))
   (no_connect (at 168.91 168.91))
+  (no_connect (at 518.16 342.9))
   (no_connect (at 495.3 39.37))
+  (no_connect (at 518.16 287.02))
+  (no_connect (at 589.28 337.82))
   (no_connect (at 427.99 524.51))
+  (no_connect (at 589.28 335.28))
   (no_connect (at -90.17 458.47))
   (no_connect (at 778.51 303.53))
@@
     (stroke (width 0) (type default))
   )
+  (wire (pts (xy 589.28 320.04) (xy 599.44 320.04))
+    (stroke (width 0) (type default))
+  )
   (wire (pts (xy 566.42 492.76) (xy 570.23 492.76))
     (stroke (width 0) (type default))
@@
     (stroke (width 0) (type default))
   )
-  (wire (pts (xy 509.27 342.9) (xy 518.16 342.9))
-    (stroke (width 0) (type default))
-  )
   (wire (pts (xy 502.92 139.7) (xy 502.92 140.97))
     (stroke (width 0) (type default))
@@
     )
   )
-  (global_label "EEP_CS" (shape output) (at 509.27 342.9 180)
-    (effects (font (size 1.27 1.27)) (justify right))
-    (property "Intersheetrefs" "${INTERSHEET_REFS}" (at 509.27 342.9 0)
+  (global_label "EEP_CS" (shape output) (at 599.44 320.04 0)
+    (effects (font (size 1.27 1.27)) (justify left))
+    (property "Intersheetrefs" "${INTERSHEET_REFS}" (at 599.44 320.04 0)
       (effects (font (size 1.27 1.27)) hide)
     )
